File: riffleito-REVC.brd (EAGLE design)
At the start: 66.8 x 18 mm, 28 parts, among them IC1 ATMEGA328P, IC2 24AA128SN, IC4 MCP1700-33, X1 16 MHz

Commit message: update
Parts:
- moved SD 0.13 mm to (33.9, 4.14)
Changed lines of the file:
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@@
 <text x="47.0916" y="17.8054" size="0.4064" layer="21" rot="R180">share your research: publiclab.org/wiki/riffle</text>
 <text x="8.6614" y="0.9906" size="0.4064" layer="22" rot="MR180">CERN Open Hardware License Ver. 1.2</text>
+<wire x1="29.337" y1="16.4592" x2="29.2862" y2="16.4592" width="0.4064" layer="21"/>
 </plain>
 <attributes>
@@
 <attribute name="NAME" x="59.3936" y="4.4734" size="0.6096" layer="25" rot="R180"/>
 </element>
-<element name="SD" library="zetex" package="SOT-23" value="FDN340P" x="33.7566" y="4.1148" smashed="yes" rot="R180">
-<attribute name="VALUE" x="35.1536" y="2.3368" size="1.27" layer="27" ratio="10" rot="R180"/>
-<attribute name="NAME" x="32.1818" y="5.0038" size="0.6096" layer="25" ratio="10"/>
+<element name="SD" library="zetex" package="SOT-23" value="FDN340P" x="33.8836" y="4.1402" smashed="yes" rot="R180">
+<attribute name="VALUE" x="35.2806" y="2.3622" size="1.27" layer="27" ratio="10" rot="R180"/>
+<attribute name="NAME" x="32.3088" y="5.0292" size="0.6096" layer="25" ratio="10"/>
 </element>
 <element name="C9" library="rcl" package="C0805@1" value=".1uF" x="41.8592" y="2.2606" smashed="yes" rot="R270">
@@
 <wire x1="33.782" y1="8.382" x2="33.6296" y2="8.4836" width="0.2032" layer="1"/>
 <wire x1="34.798" y1="6.35" x2="34.798" y2="4.064" width="0.2032" layer="1"/>
-<wire x1="34.798" y1="4.064" x2="34.798" y2="3.302" width="0.2032" layer="1"/>
-<wire x1="34.798" y1="3.302" x2="34.6964" y2="3.0988" width="0.2032" layer="1"/>
+<wire x1="34.798" y1="4.064" x2="34.8234" y2="3.1242" width="0.2032" layer="1"/>
 <wire x1="34.798" y1="6.35" x2="34.5948" y2="6.4516" width="0.2032" layer="1"/>
 <wire x1="34.798" y1="4.064" x2="36.068" y2="2.794" width="0.2032" layer="1"/>
@@
 <wire x1="18.034" y1="4.826" x2="18.542" y2="5.334" width="0.2032" layer="1"/>
 <wire x1="18.034" y1="4.064" x2="18.034" y2="4.826" width="0.2032" layer="1"/>
-<wire x1="32.766" y1="3.048" x2="32.766" y2="3.0988" width="0.2032" layer="1"/>
+<wire x1="32.766" y1="3.048" x2="32.893" y2="3.1242" width="0.2032" layer="1"/>
 <wire x1="18.034" y1="4.064" x2="18.0534" y2="3.9624" width="0.2032" layer="1"/>
 <via x="27.178" y="2.032" extent="1-16" drill="0.3302"/>
@@
 <wire x1="41.656" y1="0.508" x2="35.814" y2="0.508" width="0.2032" layer="1"/>
 <wire x1="41.656" y1="1.27" x2="41.656" y2="0.508" width="0.2032" layer="1"/>
-<wire x1="33.782" y1="5.08" x2="33.7312" y2="5.1308" width="0.2032" layer="1"/>
+<wire x1="33.782" y1="5.08" x2="33.8582" y2="5.1562" width="0.2032" layer="1"/>
 <wire x1="41.656" y1="1.27" x2="41.8592" y2="1.3106" width="0.2032" layer="1"/>
 <wire x1="41.91" y1="1.524" x2="44.704" y2="1.524" width="0.2032" layer="1"/>
