File: hardware/riffleito-REVE.sch (EAGLE design)
At the start: 28 parts, among them IC1 ATMEGA328P, IC2 24AA128SN, IC4 MCP1700-33, X1 16 MHz

Commit message: update
Parts:
- removed C9: .1uF, rcl:C-EUC0805
- removed JP4: (no value), SparkFun-Connectors:M07
- removed JP5: M10", SparkFun-Connectors:M10"
- removed S2: Reset, SparkFun:TAC_SWITCHSMD
- added CRF: 100u, resistor:C-EUC0805
- added CSD: .1uF, resistor:C-EUC0805
- added FTDI, SENSE: (no value), SparkFun-Connectors:M06SIP
- added I2C1, I2C2: 10K, rcl:R-EU_R0805
- added RAD: M04X2, SparkFun-Connectors:M04X2
- JP1: device SparkFun-Connectors:M07 -> SparkFun-Connectors:M081X08
Connections:
- net RTCINT renamed N$1
- net A0: now also SENSE.4; no longer JP4.5
- net A1: now also SENSE.5; no longer JP4.6
- net A2: now also JP1.4; no longer JP4.7
- net D10: now also RAD.3
- net D2: now also FTDI.5; no longer JP1.6
- net D3: now also JP1.5, RAD.8
- net D6: now also JP1.6; no longer JP5.8
- net D8: now also JP1.7; no longer JP5.9
- net D9: now also RAD.4
- net DTR: now also FTDI.1; no longer JP1.2
- net GND: now also CRF.2, CSD.2, FTDI.6, JP1.8, RAD.1, SENSE.1; no longer C9.1, JP1.7, JP4.4, JP5.1, JP5.10, S2.1, S2.2
- net MISO: now also RAD.7; no longer JP5.6
- net MOSI: now also RAD.6; no longer JP5.2
- net RESET: now also JP1.2; no longer JP5.4, S2.3, S2.4
- net RXD: now also FTDI.3; no longer JP1.4
- net SCK: now also RAD.5; no longer JP5.5
- net SCL: now also I2C1.2, SENSE.2; no longer JP4.1
- net SDA: now also I2C2.2, SENSE.3; no longer JP4.2
- net TXD: now also FTDI.2; no longer JP1.3
- net VCC: now also CRF.1, I2C1.1, I2C2.1, JP1.3, RAD.2, SENSE.6; no longer JP1.1, JP4.3, JP5.7
- net VDD: now also CSD.1; no longer C9.2
- net VIN: now also FTDI.4, JP1.1; no longer JP1.5, JP5.3
Other:
- note added: "i2c pullups"
- moved on the sheet: RRTC1, RTCINT
