File: hardware/riffleito-REVF-routed.sch (EAGLE design)
At the start: 31 parts, among them IC1 ATMEGA328P, IC2 24AA128SN, IC4 MCP1700-33, X1 16 MHz

Commit message: update
Changed lines of the file:
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@@
 <setting verticaltext="up"/>
 </settings>
-<grid distance="0.1" unitdist="inch" unit="inch" style="lines" multiple="1" display="no" altdistance="0.01" altunitdist="inch" altunit="inch"/>
+<grid distance="0.01" unitdist="inch" unit="inch" style="lines" multiple="1" display="no" altdistance="0.01" altunitdist="inch" altunit="inch"/>
 <layers>
 <layer number="1" name="Top" color="4" fill="1" visible="no" active="no"/>
@@
 <segment>
 <pinref part="REMOTE" gate="A" pin="D"/>
-<wire x1="-78.232" y1="15.748" x2="-80.01" y2="15.748" width="0.1524" layer="91"/>
-<wire x1="-80.01" y1="15.748" x2="-81.28" y2="15.748" width="0.1524" layer="91"/>
-<wire x1="-80.01" y1="15.748" x2="-80.01" y2="-15.24" width="0.1524" layer="91"/>
-<junction x="-80.01" y="15.748"/>
+<wire x1="-78.232" y1="15.748" x2="-80.01" y2="13.208" width="0.1524" layer="91"/>
+<wire x1="-80.01" y1="13.208" x2="-81.28" y2="15.748" width="0.1524" layer="91"/>
+<wire x1="-80.01" y1="13.208" x2="-80.01" y2="-15.24" width="0.1524" layer="91"/>
+<junction x="-80.01" y="13.208"/>
 <pinref part="C8" gate="G$1" pin="2"/>
 <pinref part="SENSE" gate="G$1" pin="6"/>
@@
 <wire x1="99.06" y1="-7.874" x2="120.65" y2="-7.874" width="0.1524" layer="91"/>
 <wire x1="120.65" y1="-7.874" x2="120.65" y2="-8.89" width="0.1524" layer="91"/>
-</segment>
-</net>
+<junction x="99.06" y="-7.874"/>
+</segment>
+</net>
