File: hardware/riffleito-REVF-routed.brd (EAGLE design)
At the start: 74.2 x 18 mm, 31 parts, among them IC1 ATMEGA328P, IC2 24AA128SN, IC4 MCP1700-33, X1 16 MHz

Commit message: update
Parts:
- moved SENSE 0.20 mm to (72.5, 2.59)
Routing:
- net VCC: track 216.0 -> 216.9 mm
Changed lines of the file:
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@@
 <attribute name="VALUE" x="42.5958" y="13.6398" size="1.27" layer="27"/>
 </element>
-<element name="SENSE" library="SparkFun-Connectors" package="1X06" value="" x="72.39" y="2.413" smashed="yes" rot="R90">
-<attribute name="VALUE" x="75.565" y="1.143" size="1.27" layer="27" rot="R90"/>
+<element name="SENSE" library="SparkFun-Connectors" package="1X06" value="" x="72.4916" y="2.5908" smashed="yes" rot="R90">
+<attribute name="VALUE" x="75.6666" y="1.3208" size="1.27" layer="27" rot="R90"/>
 </element>
 <element name="FTDI" library="SparkFun-Connectors" package="1X06" value="" x="2.1336" y="15.3162" smashed="yes" rot="R270">
@@
 <contactref element="JP2" pad="6"/>
 <contactref element="JP1" pad="10"/>
-<wire x1="72.3392" y1="2.2352" x2="68.8848" y2="2.2352" width="0.2032" layer="1"/>
+<wire x1="71.882" y1="2.2352" x2="68.8848" y2="2.2352" width="0.2032" layer="1"/>
 <wire x1="68.8848" y1="2.2352" x2="68.7832" y2="2.0456" width="0.2032" layer="1"/>
-<wire x1="72.3392" y1="2.2352" x2="72.39" y2="2.413" width="0.2032" layer="1"/>
+<wire x1="71.882" y1="2.2352" x2="72.4916" y2="2.5908" width="0.2032" layer="1"/>
 <wire x1="48.5648" y1="16.4592" x2="47.9552" y2="15.8496" width="0.2032" layer="1"/>
 <wire x1="48.5648" y1="16.6624" x2="48.5648" y2="16.4592" width="0.2032" layer="1"/>
@@
 <wire x1="47.3456" y1="2.032" x2="46.5328" y2="1.2192" width="0.2032" layer="16"/>
 <wire x1="47.3456" y1="2.032" x2="47.498" y2="2.2098" width="0.2032" layer="16"/>
-<wire x1="71.3232" y1="3.4544" x2="72.3392" y2="2.4384" width="0.2032" layer="16"/>
+<wire x1="71.3232" y1="3.4544" x2="72.4916" y2="2.6162" width="0.2032" layer="16"/>
 <wire x1="48.768" y1="3.4544" x2="71.3232" y2="3.4544" width="0.2032" layer="16"/>
 <wire x1="47.5488" y1="2.2352" x2="48.768" y2="3.4544" width="0.2032" layer="16"/>
-<wire x1="72.3392" y1="2.4384" x2="72.39" y2="2.413" width="0.2032" layer="16"/>
+<wire x1="72.4916" y1="2.6162" x2="72.4916" y2="2.5908" width="0.2032" layer="16"/>
 <wire x1="47.5488" y1="2.2352" x2="47.498" y2="2.2098" width="0.2032" layer="16"/>
 <via x="19.1008" y="1.4224" extent="1-16" drill="0.3302"/>
@@
 <wire x1="51.4096" y1="10.5664" x2="51.2064" y2="10.7696" width="0.2032" layer="16"/>
 <wire x1="71.9328" y1="10.5664" x2="51.4096" y2="10.5664" width="0.2032" layer="16"/>
-<wire x1="72.3392" y1="10.16" x2="71.9328" y2="10.5664" width="0.2032" layer="16"/>
+<wire x1="72.3392" y1="10.3378" x2="71.9328" y2="10.5664" width="0.2032" layer="16"/>
 <wire x1="20.9296" y1="10.16" x2="20.9296" y2="10.2042" width="0.2032" layer="1"/>
-<wire x1="72.3392" y1="10.16" x2="72.39" y2="10.033" width="0.2032" layer="16"/>
+<wire x1="72.3392" y1="10.3378" x2="72.4916" y2="10.2108" width="0.2032" layer="16"/>
 <via x="19.7104" y="5.2832" extent="1-16" drill="0.3302"/>
 <via x="45.9232" y="4.064" extent="1-16" drill="0.3302"/>
@@
 <wire x1="71.12" y1="6.096" x2="68.8848" y2="3.8608" width="0.2032" layer="1"/>
 <wire x1="71.12" y1="13.8176" x2="71.12" y2="6.096" width="0.2032" layer="1"/>
-<wire x1="72.3392" y1="15.0368" x2="71.12" y2="13.8176" width="0.2032" layer="1"/>
+<wire x1="72.3138" y1="15.113" x2="71.12" y2="13.8176" width="0.2032" layer="1"/>
 <wire x1="68.8848" y1="3.8608" x2="68.7832" y2="3.7456" width="0.2032" layer="1"/>
-<wire x1="72.3392" y1="15.0368" x2="72.39" y2="15.113" width="0.2032" layer="1"/>
+<wire x1="72.3138" y1="15.113" x2="72.4916" y2="15.2908" width="0.2032" layer="1"/>
 <wire x1="36.7792" y1="15.0368" x2="36.576" y2="14.8336" width="0.2032" layer="1"/>
 <wire x1="36.7792" y1="16.4592" x2="36.7792" y2="15.0368" width="0.2032" layer="1"/>
 <wire x1="37.3888" y1="17.0688" x2="36.7792" y2="16.4592" width="0.2032" layer="16"/>
 <wire x1="70.5104" y1="17.0688" x2="37.3888" y2="17.0688" width="0.2032" layer="16"/>
-<wire x1="72.3392" y1="15.24" x2="70.5104" y2="17.0688" width="0.2032" layer="16"/>
-<wire x1="72.3392" y1="15.24" x2="72.39" y2="15.113" width="0.2032" layer="16"/>
+<wire x1="72.263" y1="15.494" x2="70.5104" y2="17.0688" width="0.2032" layer="16"/>
+<wire x1="72.263" y1="15.494" x2="72.4916" y2="15.2908" width="0.2032" layer="16"/>
 <wire x1="66.04" y1="2.2352" x2="52.6288" y2="2.2352" width="0.2032" layer="1"/>
 <wire x1="66.04" y1="2.032" x2="66.04" y2="2.2352" width="0.2032" layer="1"/>
 <wire x1="67.056" y1="1.016" x2="66.04" y2="2.032" width="0.2032" layer="1"/>
 <wire x1="73.7616" y1="1.016" x2="67.056" y2="1.016" width="0.2032" layer="1"/>
-<wire x1="73.7616" y1="2.8448" x2="73.7616" y2="1.016" width="0.2032" layer="1"/>
-<wire x1="72.9488" y1="3.6576" x2="73.7616" y2="2.8448" width="0.2032" layer="1"/>
-<wire x1="68.8848" y1="3.6576" x2="72.9488" y2="3.6576" width="0.2032" layer="1"/>
+<wire x1="73.7616" y1="3.8862" x2="73.7616" y2="1.016" width="0.2032" layer="1"/>
+<wire x1="70.7898" y1="3.8862" x2="73.7616" y2="3.8862" width="0.2032" layer="1"/>
+<wire x1="68.8848" y1="3.6576" x2="70.7898" y2="3.8862" width="0.2032" layer="1"/>
 <wire x1="68.8848" y1="3.6576" x2="68.7832" y2="3.7456" width="0.2032" layer="1"/>
 <wire x1="26.6192" y1="2.8448" x2="24.9936" y2="4.4704" width="0.2032" layer="1"/>
@@
 <wire x1="36.7792" y1="17.4752" x2="35.56" y2="16.256" width="0.2032" layer="16"/>
 <wire x1="71.9328" y1="17.4752" x2="36.7792" y2="17.4752" width="0.2032" layer="16"/>
-<wire x1="74.168" y1="15.24" x2="71.9328" y2="17.4752" width="0.2032" layer="16"/>
-<wire x1="74.168" y1="12.5984" x2="74.168" y2="15.24" width="0.2032" layer="16"/>
-<wire x1="72.5424" y1="12.5984" x2="74.168" y2="12.5984" width="0.2032" layer="16"/>
+<wire x1="74.168" y1="16.4846" x2="71.9328" y2="17.4752" width="0.2032" layer="16"/>
+<wire x1="74.168" y1="12.5984" x2="74.168" y2="16.4846" width="0.2032" layer="16"/>
+<wire x1="72.6694" y1="12.7254" x2="74.168" y2="12.5984" width="0.2032" layer="16"/>
 <wire x1="20.9296" y1="11.176" x2="20.9296" y2="11.0042" width="0.2032" layer="1"/>
-<wire x1="72.5424" y1="12.5984" x2="72.39" y2="12.573" width="0.2032" layer="16"/>
+<wire x1="72.6694" y1="12.7254" x2="72.4916" y2="12.7508" width="0.2032" layer="16"/>
 <via x="22.5552" y="12.8016" extent="1-16" drill="0.3302"/>
 </signal>
@@
 <wire x1="44.2976" y1="16.0528" x2="44.1808" y2="16.1798" width="0.2032" layer="1"/>
 <wire x1="44.2976" y1="10.5664" x2="44.4754" y2="10.5248" width="0.2032" layer="1"/>
-<wire x1="71.3232" y1="8.5344" x2="72.3392" y2="7.5184" width="0.2032" layer="16"/>
+<wire x1="71.3232" y1="8.5344" x2="72.4408" y2="7.6962" width="0.2032" layer="16"/>
 <wire x1="45.9232" y1="8.5344" x2="46.5328" y2="8.5344" width="0.2032" layer="16"/>
 <wire x1="46.5328" y1="8.5344" x2="71.3232" y2="8.5344" width="0.2032" layer="16"/>
 <wire x1="44.5008" y1="9.9568" x2="45.9232" y2="8.5344" width="0.2032" layer="1"/>
 <wire x1="44.5008" y1="10.3632" x2="44.5008" y2="9.9568" width="0.2032" layer="1"/>
-<wire x1="72.3392" y1="7.5184" x2="72.39" y2="7.493" width="0.2032" layer="16"/>
+<wire x1="72.4408" y1="7.6962" x2="72.4916" y2="7.6708" width="0.2032" layer="16"/>
 <wire x1="44.5008" y1="10.3632" x2="44.4754" y2="10.5248" width="0.2032" layer="1"/>
 <wire x1="36.576" y1="7.112" x2="34.7472" y2="5.2832" width="0.2032" layer="1"/>
@@
 <wire x1="36.576" y1="2.6416" x2="36.5506" y2="2.5654" width="0.2032" layer="1"/>
 <wire x1="37.7952" y1="16.0528" x2="37.9882" y2="16.1798" width="0.2032" layer="1"/>
-<wire x1="73.7616" y1="6.2992" x2="72.5424" y2="5.08" width="0.2032" layer="1"/>
+<wire x1="73.7616" y1="6.2992" x2="72.5424" y2="5.1816" width="0.2032" layer="1"/>
 <wire x1="73.7616" y1="13.4112" x2="73.7616" y2="6.2992" width="0.2032" layer="1"/>
-<wire x1="73.3552" y1="13.8176" x2="73.7616" y2="13.4112" width="0.2032" layer="1"/>
-<wire x1="59.7408" y1="13.8176" x2="73.3552" y2="13.8176" width="0.2032" layer="16"/>
+<wire x1="73.4822" y1="13.9954" x2="73.7616" y2="13.4112" width="0.2032" layer="1"/>
+<wire x1="59.7408" y1="13.8176" x2="63.3984" y2="13.843" width="0.2032" layer="16"/>
+<wire x1="63.3984" y1="13.843" x2="63.9064" y2="13.9954" width="0.2032" layer="16"/>
+<wire x1="63.9064" y1="13.9954" x2="73.4822" y2="13.9954" width="0.2032" layer="16"/>
 <wire x1="59.3344" y1="14.224" x2="59.7408" y2="13.8176" width="0.2032" layer="16"/>
 <wire x1="43.0784" y1="14.224" x2="59.3344" y2="14.224" width="0.2032" layer="16"/>
 <wire x1="41.656" y1="12.8016" x2="43.0784" y2="14.224" width="0.2032" layer="1"/>
-<wire x1="72.5424" y1="5.08" x2="72.39" y2="4.953" width="0.2032" layer="1"/>
+<wire x1="72.5424" y1="5.1816" x2="72.4916" y2="5.1308" width="0.2032" layer="1"/>
 <via x="17.0688" y="14.6304" extent="1-16" drill="0.3302"/>
 <via x="31.0896" y="17.0688" extent="1-16" drill="0.3302"/>
-<via x="73.3552" y="13.8176" extent="1-16" drill="0.3302"/>
+<via x="73.4822" y="13.9954" extent="1-16" drill="0.3302"/>
 <via x="43.0784" y="14.224" extent="1-16" drill="0.3302"/>
 </signal>

Commit message: update
Parts:
- moved FTDI 0.59 mm to (1.55, 15.3)
Routing:
- net VIN: track 92.9 -> 93.8 mm
- net D3: track 61.4 -> 60.9 mm
- net RXD: track 14.9 -> 15.4 mm
Other:
- board size 74.2 x 18 mm -> 75 x 18.1 mm
- board text added: "A1"
- board text added: "A2"
- board text added: "D10"
- board text added: "D2"
- board text added: "D3"
- board text added: "D9"
- board text added: "DTR"
- board text added: "RXD"
- board text added: "TXD"
- board text added: "atmega328p"
- board text removed: "CERN Open Hardware License Ver. 1.2"
- board text removed: "D8"
- board text removed: "share your research: publiclab.org/wiki/riffle"

Commit message: update
Parts:
- moved CSD 0.74 mm to (68.8, 14.5)
Routing:
- net GND: track 221.9 -> 222.5 mm
Other:
- board size 75 x 18.1 mm -> 74.8 x 18 mm
- board text added: "publicab.org/wiki/riffle"
Changed lines of the file:
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@@
 <board>
 <plain>
-<wire x1="-0.254" y1="-0.0762" x2="-0.254" y2="17.9324" width="0" layer="20"/>
-<wire x1="-0.254" y1="17.9324" x2="74.7522" y2="17.9832" width="0" layer="20"/>
-<wire x1="74.7522" y1="17.9832" x2="74.7522" y2="-0.0254" width="0" layer="20"/>
-<wire x1="74.7522" y1="-0.0254" x2="-0.254" y2="-0.0762" width="0" layer="20"/>
+<wire x1="0.0762" y1="-0.0762" x2="0.0762" y2="17.9324" width="0" layer="20"/>
+<wire x1="0.0762" y1="17.9324" x2="74.9046" y2="17.9324" width="0" layer="20"/>
+<wire x1="74.9046" y1="17.9324" x2="74.9046" y2="-0.0762" width="0" layer="20"/>
+<wire x1="74.9046" y1="-0.0762" x2="0.0762" y2="-0.0762" width="0" layer="20"/>
 <text x="6.2992" y="5.207" size="0.6096" layer="21" rot="R270">ldo</text>
 <text x="41.1988" y="12.0396" size="0.6096" layer="21">EEPROM</text>
@@
 <text x="23.4442" y="14.605" size="0.6096" layer="21" rot="R180">D6</text>
 <text x="24.5618" y="13.97" size="0.6096" layer="21">GND</text>
-<text x="45.1612" y="2.9972" size="0.6096" layer="21" rot="R270">GND</text>
+<text x="45.2882" y="3.0226" size="0.6096" layer="21" rot="R270">GND</text>
 <text x="26.8478" y="6.9596" size="0.8128" layer="21" rot="R90">REV-E</text>
 <wire x1="29.337" y1="16.4592" x2="29.2862" y2="16.4592" width="0.4064" layer="21"/>
@@
 <wire x1="27.813" y1="4.8006" x2="24.0284" y2="4.8006" width="0.254" layer="21"/>
 <text x="44.9072" y="5.2578" size="0.6096" layer="21" rot="R270">D10</text>
-<text x="45.339" y="8.1026" size="0.6096" layer="21" rot="R270">SCK</text>
-<text x="45.0596" y="10.9728" size="0.6096" layer="21" rot="R270">MISO</text>
-<text x="45.1358" y="13.9954" size="0.6096" layer="21" rot="R270">RESET</text>
-<text x="51.5366" y="12.5984" size="0.6096" layer="21" rot="R270">VIN</text>
-<text x="51.6382" y="10.2616" size="0.6096" layer="21" rot="R270">D3</text>
-<text x="51.4858" y="8.4328" size="0.6096" layer="21" rot="R270">MOSI</text>
+<text x="45.4152" y="8.001" size="0.6096" layer="21" rot="R270">SCK</text>
+<text x="45.3644" y="11.2014" size="0.6096" layer="21" rot="R270">MISO</text>
+<text x="45.339" y="14.4526" size="0.6096" layer="21" rot="R270">RESET</text>
+<text x="51.562" y="12.573" size="0.6096" layer="21" rot="R270">VIN</text>
+<text x="51.562" y="10.2616" size="0.6096" layer="21" rot="R270">D3</text>
+<text x="51.5366" y="8.3566" size="0.6096" layer="21" rot="R270">MOSI</text>
 <text x="51.5366" y="5.3848" size="0.6096" layer="21" rot="R270">D9</text>
 <text x="51.5112" y="3.8608" size="0.6096" layer="21" rot="R270">3.3V</text>
@@
 <text x="3.5306" y="1.905" size="0.6096" layer="21" rot="R90">GND</text>
 <text x="18.9484" y="9.6774" size="0.6096" layer="21" rot="R216">atmega328p</text>
+<text x="28.9306" y="0.381" size="0.6096" layer="21">publicab.org/wiki/riffle</text>
 </plain>
 <attributes>
@@
 </element>
 <element name="MICROSD" library="adafruit" package="MICROSD" value="MICROSD" x="66.675" y="0.762" smashed="yes" rot="R180">
-<attribute name="NAME" x="58.5046" y="4.8798" size="0.8128" layer="25" rot="R180"/>
+<attribute name="NAME" x="61.324" y="5.1592" size="0.6096" layer="25" rot="R180"/>
 </element>
 <element name="SD" library="zetex" package="SOT-23" value="FDN340P" x="24.5364" y="11.811" smashed="yes" rot="R180">
@@
 <attribute name="VALUE" x="30.3212" y="18.0086" size="0.4064" layer="27" rot="R180"/>
 </element>
-<element name="CSD" library="resistor" package="C0805" value=".1uF" x="68.7578" y="15.24" smashed="yes" rot="R90">
-<attribute name="NAME" x="67.0814" y="17.0688" size="0.6096" layer="25" rot="R270"/>
-<attribute name="VALUE" x="71.0438" y="14.351" size="1.27" layer="27" rot="R90"/>
+<element name="CSD" library="resistor" package="C0805" value=".1uF" x="68.8086" y="14.5034" smashed="yes" rot="R90">
+<attribute name="NAME" x="67.1322" y="16.3322" size="0.6096" layer="25" rot="R270"/>
+<attribute name="VALUE" x="71.0946" y="13.6144" size="1.27" layer="27" rot="R90"/>
 </element>
 <element name="JP2" library="SparkFun-Connectors" package="1X06_LOCK" value="" x="12.573" y="16.3068" smashed="yes">
@@
 <wire x1="48.5648" y1="16.4592" x2="47.9552" y2="15.8496" width="0.2032" layer="1"/>
 <wire x1="48.5648" y1="16.6624" x2="48.5648" y2="16.4592" width="0.2032" layer="1"/>
-<wire x1="48.9712" y1="17.0688" x2="48.5648" y2="16.6624" width="0.2032" layer="1"/>
-<wire x1="53.0352" y1="17.0688" x2="48.9712" y2="17.0688" width="0.2032" layer="1"/>
+<wire x1="48.9712" y1="16.9672" x2="48.5648" y2="16.6624" width="0.2032" layer="1"/>
+<wire x1="53.0352" y1="16.9672" x2="48.9712" y2="16.9672" width="0.2032" layer="1"/>
 <wire x1="53.0352" y1="15.24" x2="53.0352" y2="15.8496" width="0.2032" layer="1"/>
-<wire x1="53.0352" y1="15.8496" x2="53.0352" y2="17.0688" width="0.2032" layer="1"/>
+<wire x1="53.0352" y1="15.8496" x2="53.0352" y2="16.9672" width="0.2032" layer="1"/>
 <wire x1="47.9552" y1="15.8496" x2="47.9434" y2="15.8496" width="0.2032" layer="1"/>
 <wire x1="53.0352" y1="15.24" x2="53.075" y2="15.202" width="0.2032" layer="1"/>
@@
 <wire x1="63.1952" y1="11.9888" x2="63.175" y2="11.802" width="0.2032" layer="1"/>
 <wire x1="66.2432" y1="14.224" x2="66.275" y2="14.302" width="0.2032" layer="1"/>
-<wire x1="66.4464" y1="16.0528" x2="68.6816" y2="16.0528" width="0.2032" layer="1"/>
+<wire x1="66.4464" y1="16.0528" x2="68.834" y2="16.0528" width="0.2032" layer="1"/>
 <wire x1="66.4464" y1="14.4272" x2="66.4464" y2="16.0528" width="0.2032" layer="1"/>
-<wire x1="68.6816" y1="16.0528" x2="68.7578" y2="16.09" width="0.2032" layer="1"/>
+<wire x1="68.834" y1="16.0528" x2="68.8086" y2="15.3534" width="0.2032" layer="1"/>
 <wire x1="66.4464" y1="14.4272" x2="66.275" y2="14.302" width="0.2032" layer="1"/>
 <wire x1="56.896" y1="15.8496" x2="53.0352" y2="15.8496" width="0.2032" layer="1"/>
@@
 <wire x1="41.2496" y1="14.0208" x2="39.2176" y2="14.0208" width="0.2032" layer="16"/>
 <wire x1="41.2496" y1="17.0688" x2="41.2496" y2="14.0208" width="0.2032" layer="1"/>
-<wire x1="41.656" y1="17.4752" x2="41.2496" y2="17.0688" width="0.2032" layer="1"/>
-<wire x1="58.7248" y1="17.4752" x2="41.656" y2="17.4752" width="0.2032" layer="1"/>
-<wire x1="58.7248" y1="11.176" x2="58.7248" y2="17.4752" width="0.2032" layer="1"/>
+<wire x1="41.6814" y1="17.399" x2="41.2496" y2="17.0688" width="0.2032" layer="1"/>
+<wire x1="58.7248" y1="17.399" x2="41.6814" y2="17.399" width="0.2032" layer="1"/>
+<wire x1="58.7248" y1="11.176" x2="58.7248" y2="17.399" width="0.2032" layer="1"/>
 <wire x1="15.4432" y1="4.064" x2="15.437" y2="3.9116" width="0.2032" layer="1"/>
 <wire x1="58.7248" y1="11.176" x2="58.775" y2="11.002" width="0.2032" layer="1"/>
 <wire x1="70.3072" y1="11.176" x2="68.8848" y2="9.7536" width="0.2032" layer="1"/>
 <wire x1="70.3072" y1="17.0688" x2="70.3072" y2="11.176" width="0.2032" layer="1"/>
-<wire x1="69.9008" y1="17.4752" x2="70.3072" y2="17.0688" width="0.2032" layer="1"/>
-<wire x1="58.7248" y1="17.4752" x2="69.9008" y2="17.4752" width="0.2032" layer="1"/>
+<wire x1="69.9008" y1="17.4244" x2="70.3072" y2="17.0688" width="0.2032" layer="1"/>
+<wire x1="58.7248" y1="17.399" x2="69.9008" y2="17.4244" width="0.2032" layer="1"/>
 <wire x1="68.8848" y1="9.7536" x2="68.7578" y2="9.6926" width="0.2032" layer="1"/>
 <via x="15.4432" y="8.128" extent="1-16" drill="0.3302"/>
@@
 <contactref element="MICROSD" pad="4"/>
 <contactref element="CSD" pad="1"/>
-<wire x1="68.8848" y1="14.224" x2="68.8848" y2="11.7856" width="0.2032" layer="1"/>
+<wire x1="68.8848" y1="14.224" x2="68.8848" y2="13.6652" width="0.2032" layer="1"/>
+<wire x1="68.8848" y1="13.6652" x2="68.8848" y2="11.7856" width="0.2032" layer="1"/>
 <wire x1="68.8848" y1="11.7856" x2="68.7578" y2="11.5926" width="0.2032" layer="1"/>
-<wire x1="68.8848" y1="14.224" x2="68.7578" y2="14.39" width="0.2032" layer="1"/>
+<wire x1="68.8848" y1="14.224" x2="68.8086" y2="13.6534" width="0.2032" layer="1"/>
 <wire x1="26.416" y1="13.0048" x2="24.5872" y2="13.0048" width="0.2032" layer="1"/>
 <wire x1="26.6192" y1="13.208" x2="26.416" y2="13.0048" width="0.2032" layer="16"/>
@@
 <wire x1="24.5872" y1="13.0048" x2="24.511" y2="12.827" width="0.2032" layer="1"/>
 <wire x1="60.96" y1="11.9888" x2="60.975" y2="11.802" width="0.2032" layer="1"/>
-<wire x1="69.9008" y1="14.4272" x2="68.8848" y2="14.4272" width="0.2032" layer="1"/>
-<wire x1="69.9008" y1="16.8656" x2="69.9008" y2="14.4272" width="0.2032" layer="1"/>
-<wire x1="69.6976" y1="17.0688" x2="69.9008" y2="16.8656" width="0.2032" layer="1"/>
-<wire x1="61.1632" y1="17.0688" x2="69.6976" y2="17.0688" width="0.2032" layer="1"/>
-<wire x1="61.1632" y1="11.9888" x2="61.1632" y2="17.0688" width="0.2032" layer="1"/>
-<wire x1="68.8848" y1="14.4272" x2="68.7578" y2="14.39" width="0.2032" layer="1"/>
+<wire x1="69.9008" y1="13.6652" x2="68.8848" y2="13.6652" width="0.2032" layer="1"/>
+<wire x1="69.9008" y1="16.5354" x2="69.9008" y2="13.6652" width="0.2032" layer="1"/>
+<wire x1="69.6976" y1="16.637" x2="69.9008" y2="16.5354" width="0.2032" layer="1"/>
+<wire x1="61.1632" y1="16.637" x2="69.6976" y2="16.637" width="0.2032" layer="1"/>
+<wire x1="61.1632" y1="11.9888" x2="61.1632" y2="16.637" width="0.2032" layer="1"/>
+<wire x1="68.8848" y1="13.6652" x2="68.8086" y2="13.6534" width="0.2032" layer="1"/>
 <wire x1="61.1632" y1="11.9888" x2="60.975" y2="11.802" width="0.2032" layer="1"/>
 <via x="26.416" y="13.0048" extent="1-16" drill="0.3302"/>
