File: hardware/riffleito-REVG.brd (EAGLE design)
At the start: 74.8 x 18 mm, 31 parts, among them IC1 ATMEGA328P, IC2 24AA128SN, IC4 MCP1700-33, X1 16 MHz

Commit message: update
Routing:
- net RXD: track 18.9 -> 20.2 mm
Other:
- board text added: "D8"
Changed lines of the file:
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@@
 <wire x1="74.9046" y1="17.9324" x2="74.9046" y2="-0.0762" width="0" layer="20"/>
 <wire x1="74.9046" y1="-0.0762" x2="0.0762" y2="-0.0762" width="0" layer="20"/>
-<text x="6.2992" y="5.207" size="0.6096" layer="21" rot="R270">ldo</text>
+<text x="6.3246" y="4.3434" size="0.6096" layer="21" rot="R270">ldo</text>
 <text x="41.1988" y="12.0396" size="0.6096" layer="21">EEPROM</text>
-<text x="13.97" y="14.1986" size="0.6096" layer="21">A2</text>
-<text x="13.6398" y="14.6304" size="0.6096" layer="21" rot="R180">3.3V</text>
-<text x="18.6436" y="14.5288" size="0.6096" layer="21" rot="R180">D3</text>
-<text x="20.828" y="14.6304" size="0.6096" layer="21" rot="R180">D6</text>
-<text x="23.4442" y="14.605" size="0.6096" layer="21" rot="R180">D6</text>
-<text x="24.5618" y="13.97" size="0.6096" layer="21">GND</text>
+<text x="22.606" y="13.6144" size="0.6096" layer="21">A1</text>
+<text x="26.7716" y="14.0716" size="0.6096" layer="21" rot="R180">3.3V</text>
+<text x="18.3388" y="14.1478" size="0.6096" layer="21" rot="R180">D3</text>
+<text x="13.3604" y="14.1732" size="0.6096" layer="21" rot="R180">D8</text>
+<text x="15.9258" y="14.1732" size="0.6096" layer="21" rot="R180">D6</text>
+<text x="9.4488" y="13.716" size="0.6096" layer="21">GND</text>
 <text x="45.212" y="3.175" size="0.6096" layer="21" rot="R270">GND</text>
 <wire x1="29.337" y1="16.4592" x2="29.2862" y2="16.4592" width="0.4064" layer="21"/>
 <text x="44.8818" y="5.461" size="0.6096" layer="21" rot="R270">D10</text>
-<text x="45.4152" y="8.001" size="0.6096" layer="21" rot="R270">SCK</text>
-<text x="45.3644" y="11.2014" size="0.6096" layer="21" rot="R270">MISO</text>
+<text x="45.1866" y="8.3312" size="0.6096" layer="21" rot="R270">SCK</text>
+<text x="45.085" y="11.0744" size="0.6096" layer="21" rot="R270">MISO</text>
 <text x="45.339" y="14.4526" size="0.6096" layer="21" rot="R270">RESET</text>
 <text x="51.562" y="12.573" size="0.6096" layer="21" rot="R270">VIN</text>
-<text x="51.562" y="10.2616" size="0.6096" layer="21" rot="R270">D3</text>
-<text x="51.5366" y="8.3566" size="0.6096" layer="21" rot="R270">MOSI</text>
-<text x="51.5366" y="5.3848" size="0.6096" layer="21" rot="R270">D9</text>
-<text x="51.689" y="3.8608" size="0.6096" layer="21" rot="R270">3.3V</text>
+<text x="51.7652" y="10.3378" size="0.6096" layer="21" rot="R270">D3</text>
+<text x="51.7144" y="8.4074" size="0.6096" layer="21" rot="R270">MOSI</text>
+<text x="51.7144" y="5.4102" size="0.6096" layer="21" rot="R270">D9</text>
+<text x="51.816" y="3.3274" size="0.6096" layer="21" rot="R270">3.3V</text>
 <text x="70.4596" y="16.4592" size="0.6096" layer="21" rot="R270">3.3V</text>
-<text x="70.3072" y="13.335" size="0.6096" layer="21" rot="R270">A1</text>
+<text x="70.3072" y="13.335" size="0.6096" layer="21" rot="R270">D2</text>
 <text x="70.4342" y="10.8966" size="0.6096" layer="21" rot="R270">A1</text>
 <text x="70.4342" y="8.7884" size="0.6096" layer="21" rot="R270">SDA</text>
@@
 <text x="70.5358" y="3.3528" size="0.6096" layer="21" rot="R270">GND</text>
 <text x="3.3274" y="14.7574" size="0.6096" layer="21" rot="R90">DTR</text>
-<text x="3.3528" y="12.1412" size="0.6096" layer="21" rot="R90">TXD</text>
+<text x="3.5052" y="11.938" size="0.6096" layer="21" rot="R90">TXD</text>
 <text x="3.4036" y="9.398" size="0.6096" layer="21" rot="R90">RXD</text>
 <text x="3.4544" y="6.9342" size="0.6096" layer="21" rot="R90">VIN</text>
-<text x="3.4544" y="4.2418" size="0.6096" layer="21" rot="R90">D2</text>
+<text x="3.5306" y="4.445" size="0.6096" layer="21" rot="R90">GND</text>
 <text x="3.5306" y="1.905" size="0.6096" layer="21" rot="R90">GND</text>
 <text x="18.9484" y="9.6774" size="0.6096" layer="21" rot="R216">atmega328p</text>
 <text x="69.5452" y="3.2512" size="0.8128" layer="22" rot="MR0">publicab.org/wiki/riffle</text>
-<text x="34.671" y="0.3302" size="0.8128" layer="21">RIFFLE-ITO REV-F</text>
+<text x="31.5468" y="0.2032" size="0.8128" layer="21">RIFFLE-ITO REV-F</text>
 <text x="69.596" y="4.445" size="0.8128" layer="22" rot="MR0">RIFFLE-IT REV-F</text>
 <text x="69.2658" y="1.778" size="0.8128" layer="22" rot="MR0">CERN OHL v1.2</text>
@@
 <wire x1="74.3712" y1="0.6858" x2="44.7294" y2="0.6604" width="0.4064" layer="22"/>
 <wire x1="44.7294" y1="0.6604" x2="44.7294" y2="14.9098" width="0.4064" layer="22"/>
-<text x="65.278" y="9.0424" size="0.8128" layer="22" rot="MR0">&lt;&lt;nordic RF24&gt;&gt;</text>
+<text x="66.4972" y="13.462" size="0.8128" layer="22" rot="MR0">&lt;&lt;nordic RF24&gt;&gt;</text>
 <text x="45.7454" y="3.2004" size="0.6096" layer="22" rot="MR270">GND</text>
 <wire x1="46.1264" y1="0.6604" x2="46.1264" y2="11.176" width="0.4064" layer="22"/>
 <wire x1="51.7144" y1="0.635" x2="51.7144" y2="10.9474" width="0.4064" layer="22"/>
 <wire x1="51.6382" y1="11.1252" x2="46.101" y2="11.1506" width="0.4064" layer="22"/>
+<text x="19.8374" y="13.462" size="0.6096" layer="21">A2</text>
 </plain>
 <attributes>
@@
 </element>
 <element name="X1" library="SparkFun" package="RESONATOR-SMD" value="16 MHz" x="8.9916" y="6.7818" smashed="yes" rot="R270">
-<attribute name="NAME" x="10.1092" y="8.255" size="0.6096" layer="25"/>
+<attribute name="NAME" x="10.1346" y="7.5438" size="0.6096" layer="25"/>
 <attribute name="VALUE" x="7.4676" y="7.6708" size="0.4064" layer="27" rot="R270"/>
 </element>
@@
 <element name="BAT" library="SparkFunNew" package="BATTCON_12MM_SMT" value="CR1220" x="38.6334" y="8.4836" rot="MR270"/>
 <element name="RRST" library="rcl" package="R0805" value="10K" x="9.2202" y="12.7762" smashed="yes">
-<attribute name="NAME" x="10.9728" y="14.1986" size="0.6096" layer="25" rot="R270"/>
+<attribute name="NAME" x="9.525" y="11.176" size="0.6096" layer="25"/>
 <attribute name="VALUE" x="8.5852" y="10.2362" size="1.27" layer="27"/>
 </element>
@@
 </element>
 <element name="RM2" library="rcl" package="R0805" value="10K" x="12.1158" y="1.3716" smashed="yes">
-<attribute name="NAME" x="13.6652" y="2.8702" size="0.6096" layer="25" rot="R180"/>
+<attribute name="NAME" x="13.081" y="2.9718" size="0.6096" layer="25" rot="R180"/>
 <attribute name="VALUE" x="11.4808" y="-1.1684" size="1.27" layer="27"/>
 </element>
@@
 <attribute name="VALUE" x="51.562" y="7.0358" size="0.4064" layer="28" font="vector" rot="MR90"/>
 </element>
-<element name="JP3" library="SparkFun-Connectors" package="1X07" value="" x="25.4762" y="15.8242" rot="R180"/>
+<element name="JP3" library="SparkFun-Connectors" package="1X07" value="" x="25.4762" y="15.8242" smashed="yes" rot="R180">
+<attribute name="VALUE" x="26.7462" y="18.9992" size="1.27" layer="27" rot="R180"/>
+</element>
 </elements>
 <signals>
@@
 <wire x1="5.08" y1="11.7856" x2="14.0208" y2="11.7856" width="0.2032" layer="16"/>
 <wire x1="3.4544" y1="13.4112" x2="5.08" y2="11.7856" width="0.2032" layer="16"/>
-<wire x1="3.048" y1="13.4112" x2="3.4544" y2="13.4112" width="0.2032" layer="16"/>
-<wire x1="2.8448" y1="13.208" x2="3.048" y2="13.4112" width="0.2032" layer="1"/>
+<wire x1="2.9718" y1="14.224" x2="3.4544" y2="13.4112" width="0.2032" layer="16"/>
+<wire x1="2.8448" y1="13.208" x2="2.9718" y2="14.224" width="0.2032" layer="1"/>
 <wire x1="2.8448" y1="12.192" x2="2.8448" y2="13.208" width="0.2032" layer="1"/>
 <wire x1="1.6256" y1="10.9728" x2="2.8448" y2="12.192" width="0.2032" layer="1"/>
@@
 <wire x1="1.6256" y1="10.3632" x2="1.5494" y2="10.1854" width="0.2032" layer="1"/>
 <via x="15.6464" y="11.176" extent="1-16" drill="0.3302"/>
-<via x="3.048" y="13.4112" extent="1-16" drill="0.3302"/>
+<via x="2.9718" y="14.224" extent="1-16" drill="0.3302"/>
 </signal>
 <signal name="TXD">
@@
 <wire x1="4.8768" y1="1.6256" x2="4.8158" y2="1.4478" width="0.381" layer="1"/>
 <wire x1="3.4544" y1="12.3952" x2="4.2672" y2="13.208" width="0.381" layer="1"/>
-<wire x1="3.4544" y1="11.7856" x2="3.4544" y2="12.3952" width="0.381" layer="1"/>
-<wire x1="3.4544" y1="7.7216" x2="3.4544" y2="11.7856" width="0.381" layer="16"/>
+<wire x1="3.4544" y1="11.4554" x2="3.4544" y2="12.3952" width="0.381" layer="1"/>
+<wire x1="3.4544" y1="7.7216" x2="3.4544" y2="11.4554" width="0.381" layer="16"/>
 <wire x1="1.6256" y1="7.7216" x2="3.4544" y2="7.7216" width="0.381" layer="16"/>
 <wire x1="4.2672" y1="13.208" x2="4.4586" y2="13.2334" width="0.381" layer="1"/>
@@
 <wire x1="50.1904" y1="12.3952" x2="50.038" y2="12.3698" width="0.381" layer="16"/>
 <wire x1="4.2672" y1="13.4112" x2="4.4586" y2="13.2334" width="0.381" layer="1"/>
-<via x="3.4544" y="11.7856" extent="1-16" drill="0.3302"/>
+<via x="3.4544" y="11.4554" extent="1-16" drill="0.3302"/>
 <via x="4.2672" y="4.8768" extent="1-16" drill="0.3302"/>
 <via x="53.6448" y="12.3952" extent="1-16" drill="0.3302"/>

Commit message: update
Parts:
- moved SENSE 0.69 mm to (71.8, 2.39)
Routing:
- net GND: track 255.9 -> 254.6 mm
- net A0: track 55.4 -> 54.7 mm
- net D2: track 61.3 -> 60.6 mm
- net SCL: track 115.6 -> 115.0 mm
- net SDA: track 89.4 -> 88.8 mm
- net VCC: track 167.0 -> 166.5 mm
Other:
- board size 74.8 x 18 mm -> 73.7 x 18.1 mm
