File: hardware/riffleito-REVD.brd (EAGLE design)
At the start: 66.8 x 18 mm, 29 parts, among them IC1 ATMEGA328P, IC2 24AA128SN, IC4 MCP1700-33, X1 16 MHz

Commit message: routed!
Parts:
- moved RAD 38.6 mm to (48.2, 8.38), turned to 90 degrees
- moved C7 14.7 mm to (5.84, 16.0), turned to 0 degrees
- moved RSD1 13.3 mm to (47.1, 15.4), turned to 0 degrees
- moved SENSE 12.9 mm to (67.8, 15.3), turned to 270 degrees
- moved X1 8.93 mm to (10.4, 6.86), turned to 270 degrees
- moved SD 8.78 mm to (42.5, 1.91), turned to 90 degrees
- moved BAT 7.25 mm to (38.7, 8.79)
- moved REMOTE 6.33 mm to (23.9, 2.21), turned to 90 degrees
- moved C9 5.78 mm to (47.6, 1.40), turned to 0 degrees
- moved C3 5.18 mm to (9.17, 10.3), turned to 180 degrees
- moved C6 4.38 mm to (10.3, 2.31)
- moved JP2 4.25 mm to (9.68, 16.2)
- moved MICROSD 4.20 mm to (65.8, 0.99)
- moved RRST 4.13 mm to (9.78, 13.0), turned to 0 degrees
- moved C4 3.71 mm to (18.2, 1.32)
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Connections:
- net A0: now also SENSE.4; no longer SENSE.5
- net A1: now also SENSE.5; no longer SENSE.6
- net GND: now also SENSE.1; no longer SENSE.4
- net SCL: now also SENSE.2; no longer SENSE.1
- net SDA: now also SENSE.3; no longer SENSE.2
- net VCC: now also SENSE.6; no longer SENSE.3
Routing:
- net GND: track 0.00 -> 184.0 mm, vias 0 -> 7
- net VCC: track 0.00 -> 134.8 mm, vias 0 -> 10
- net SCL: track 0.00 -> 71.4 mm, vias 0 -> 4
- net SDA: track 0.00 -> 67.8 mm, vias 0 -> 3
- net D7: track 0.00 -> 66.2 mm, vias 0 -> 2
- net A1: track 0.00 -> 56.0 mm, vias 0 -> 2
- net MISO: track 0.00 -> 54.6 mm, vias 0 -> 3
- net A0: track 0.00 -> 53.3 mm, vias 0 -> 3
- net MOSI: track 0.00 -> 48.4 mm, vias 0 -> 4
- net D3: track 0.00 -> 44.5 mm, vias 0 -> 4
- net SCK: track 0.00 -> 43.9 mm, vias 0 -> 2
- net VDD: track 0.00 -> 42.3 mm, vias 0 -> 2
- net D10: track 0.00 -> 38.7 mm, vias 0 -> 2
- net D5: track 0.00 -> 28.4 mm, vias 0 -> 2
- net D9: track 0.00 -> 27.4 mm, vias 0 -> 2
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Other:
- board size 66.8 x 18 mm -> 68.7 x 18 mm

Commit message: update
Parts:
- moved I2C1 1.45 mm to (31.1, 14.0)
- moved I2C2 1.40 mm to (31.0, 16.4)
- moved RRTC1 1.35 mm to (36.8, 2.01)
- moved RSD1 1.21 mm to (48.2, 15.7)
- moved C4 0.91 mm to (19.2, 1.32)
- moved C10 0.67 mm to (6.02, 9.55)
- moved C9 0.66 mm to (48.2, 1.45)
- moved REMOTE 0.48 mm to (24.4, 2.24)
- moved C5 0.41 mm to (29.1, 1.19)
- moved RM2 0.39 mm to (14.2, 1.30)
- moved C6 0.32 mm to (10.6, 2.21)
- moved IC4 0.31 mm to (7.09, 4.93)
- moved MICROSD 0.26 mm to (65.8, 0.74)
- moved RM1 0.20 mm to (7.04, 1.42)
- moved IC1 0.18 mm to (17.9, 8.53)
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Routing:
- net VCC: track 134.8 -> 200.2 mm, vias 10 -> 11
- net MOSI: track 48.4 -> 67.3 mm, vias 4 -> 3
- net D7: track 66.2 -> 52.8 mm, vias 2 -> 3
- net D6: track 16.8 -> 30.1 mm, vias 1 -> 3
- net A3: track 22.2 -> 32.4 mm, vias 2 -> 4
- net D8: track 23.1 -> 13.9 mm, vias 4 -> 0
- net D3: track 44.5 -> 52.2 mm, vias 4 -> 3
- net D4: track 20.7 -> 28.3 mm, vias 2 -> 4
- net SCK: track 43.9 -> 50.8 mm, vias 2 -> 3
- net D10: track 38.7 -> 32.4 mm, vias 2 -> 1
- net MISO: track 54.6 -> 60.8 mm, vias 3 -> 5
- net A0: track 53.3 -> 57.9 mm
- net GND: track 184.0 -> 179.6 mm, vias 7 -> 5
- net RESET: track 21.0 -> 16.9 mm, vias 2 -> 1
- net D2: track 16.0 -> 19.0 mm
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
Commit message: update - routed
Parts:
- moved JP2 1.68 mm to (11.4, 16.2)
- moved C7 1.54 mm to (7.19, 15.2)
- moved C3 0.65 mm to (9.80, 10.2)
- moved RRST 0.51 mm to (10.2, 12.7)
- moved C10 0.14 mm to (6.12, 9.65)
- moved C1 0.11 mm to (6.02, 12.7)
Routing:
- net SDA: track 68.4 -> 106.6 mm, vias 3 -> 6
- net VCC: track 200.2 -> 176.2 mm, vias 11 -> 9
- net GND: track 179.6 -> 200.8 mm, vias 5 -> 7
- net MOSI: track 67.3 -> 49.0 mm
- net D6: track 30.1 -> 17.4 mm, vias 3 -> 1
- net D9: track 27.5 -> 39.0 mm
- net D4: track 28.3 -> 18.0 mm, vias 4 -> 2
- net D7: track 52.8 -> 63.1 mm, vias 3 -> 4
- net A0: track 57.9 -> 47.8 mm, vias 3 -> 1
- net A3: track 32.4 -> 23.1 mm
- net D3: track 52.2 -> 44.7 mm, vias 3 -> 2
- net MISO: track 60.8 -> 53.7 mm, vias 5 -> 4
- net VDD: track 41.9 -> 34.9 mm
- net D10: track 32.4 -> 39.4 mm, vias 1 -> 4
- net D8: track 13.9 -> 18.5 mm, vias 0 -> 2
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
Commit message: update
Changed lines of the file:
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@@
 <plain>
 <wire x1="0.5842" y1="-0.0254" x2="0.5842" y2="17.9832" width="0" layer="20"/>
-<wire x1="0.5842" y1="17.9832" x2="69.3166" y2="18.0086" width="0" layer="20"/>
-<wire x1="69.3166" y1="18.0086" x2="69.3166" y2="0" width="0" layer="20"/>
-<wire x1="69.3166" y1="0" x2="0.5842" y2="-0.0254" width="0" layer="20"/>
+<wire x1="0.5842" y1="17.9832" x2="69.2404" y2="18.0086" width="0" layer="20"/>
+<wire x1="69.2404" y1="18.0086" x2="69.2404" y2="0" width="0" layer="20"/>
+<wire x1="69.2404" y1="0" x2="0.5842" y2="-0.0254" width="0" layer="20"/>
 <text x="4.2418" y="5.0038" size="0.6096" layer="21" rot="R90">ldo</text>
 <text x="29.8196" y="13.3604" size="0.6096" layer="21" rot="R270">EEPROM</text>

Commit message: update
Parts:
- removed C9: .1uF, rcl:C0805@1
- removed FTDI, SENSE: (no value), SparkFun-Connectors:1X06
- removed RAD: M04X2, SparkFun-Connectors:2X4
- added CRF: 100u, resistor:C0805
- added CSD: .1uF, resistor:C0805
- added JP1: (no value), SparkFun-Connectors:1X08
- added JP4: (no value), SparkFun-Connectors:1X07
- added RTCINT: SOLDERJUMPERNO, _SparkFun:SJ_2S-NO
- added U$1: M04X2, SparkFun-Connectors:2X4
- JP2: device SparkFun-Connectors:1X07 -> SparkFun-Connectors:1X06
- moved C8 42.2 mm to (69.2, 16.5), turned to 180 degrees
- moved RRTC1 15.0 mm to (31.7, 16.1), turned to 180 degrees
- moved I2C1 14.4 mm to (39.2, 2.08)
- moved SD 13.6 mm to (44.2, 15.4), turned to 180 degrees
- moved JP2 9.86 mm to (1.52, 15.4), turned to 270 degrees
- moved RTC 9.09 mm to (31.0, 6.99), turned to 180 degrees
- moved IC2 8.93 mm to (40.1, 8.31), turned to 0 degrees
- moved I2C2 8.90 mm to (39.9, 16.0)
- moved C5 7.94 mm to (24.0, 7.29), turned to 270 degrees
- moved C4 2.36 mm to (16.8, 1.40)
- moved RM2 2.13 mm to (12.1, 1.37)
- moved C7 2.01 mm to (5.61, 16.4)
- moved IC4 1.64 mm to (5.46, 5.11)
- moved C6 1.60 mm to (9.02, 2.29)
- moved C3 1.60 mm to (8.20, 10.2)
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Connections:
- new net N$1: RRTC1.2, RTC.3, RTCINT.1
- new net N$4: JP4.7, REMOTE.1
- net A0: now also JP4.2; no longer SENSE.4
- net A1: now also JP4.3; no longer SENSE.5
- net A2: now also JP1.4; no longer JP2.4
- net D10: now also U$1.6; no longer RAD.3
- net D2: now also JP4.4; no longer FTDI.5
- net D3: now also JP1.5, RTCINT.2, U$1.1; no longer RAD.4
- net D6: now also JP1.6; no longer JP2.5
- net D8: now also JP1.7; no longer JP2.6
- net D9: now also U$1.5; no longer RRTC1.2, RTC.3
- net DTR: now also JP2.1; no longer FTDI.1
- net GND: now also CRF.2, CSD.2, JP1.8, JP2.5, JP2.6, JP4.1, U$1.8; no longer C9.1, FTDI.6, JP2.7, RAD.1, SENSE.1
- net MISO: now also U$1.2; no longer RAD.7
- net MOSI: now also U$1.3; no longer RAD.6
- net RESET: now also JP1.2; no longer JP2.2
- net RXD: now also JP2.3; no longer FTDI.3
- net SCK: now also U$1.4; no longer RAD.5
- net SCL: now also JP4.6; no longer SENSE.2
- net SDA: now also JP4.5; no longer SENSE.3
- net TXD: now also JP2.2; no longer FTDI.2
- net VCC: now also CRF.1, JP1.3, U$1.7; no longer C8.2, JP2.3, RAD.2, REMOTE.1, SENSE.6
- net VDD: now also CSD.1; no longer C9.2
- net VIN: now also JP1.1, JP2.4; no longer FTDI.4, JP2.1
Routing:
- net N$4: track 0.00 -> 65.2 mm, vias 0 -> 3
- net D2: track 16.5 -> 70.5 mm, vias 1 -> 5
- net VCC: track 176.2 -> 151.4 mm, vias 9 -> 8
- net D3: track 44.7 -> 66.4 mm, vias 2 -> 5
- net SDA: track 106.6 -> 85.3 mm, vias 6 -> 8
- net N$1: track 0.00 -> 15.1 mm
- net AREF: track 17.5 -> 3.89 mm, vias 2 -> 0
- net SCL: track 71.2 -> 83.5 mm, vias 4 -> 5
- net A0: track 47.8 -> 60.0 mm, vias 1 -> 3
- net D4: track 18.0 -> 28.5 mm, vias 2 -> 4
- net VDD: track 34.9 -> 25.4 mm
- net A1: track 57.2 -> 65.4 mm
- net D5: track 29.1 -> 37.3 mm
- net RTC_BATT: track 9.82 -> 17.2 mm
- net D7: track 63.1 -> 70.1 mm, vias 4 -> 2
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Other:
- board size 68.7 x 18 mm -> 74.9 x 18 mm
- board text added: "<<nordic RF24>>"
- board text added: "CERN OHL v1.2"
- board text added: "D10"
- board text added: "D3"
- board text added: "D9"
- board text added: "RIFFLE-IT REV-F"
- board text added: "RIFFLE-ITO REV-F"
- board text added: "atmega328p"
- board text added: "publicab.org/wiki/riffle"
- board text removed: "A0"
- board text removed: "CERN Open Hardware License Ver. 1.2"
- board text removed: "REV-C"
- board text removed: "riffle-ito"
- board text removed: "share your research: publiclab.org/wiki/riffle"

Commit message: update
Parts:
- moved C8 0.74 mm to (69.1, 15.8), turned to 90 degrees
Connections:
- net N$4: now also C8.2
Routing:
- net MOSI: track 47.6 -> 69.0 mm, vias 2 -> 3
- net SDA: track 85.3 -> 101.8 mm, vias 8 -> 7
- net D3: track 66.4 -> 79.2 mm, vias 5 -> 6
- net D4: track 28.5 -> 16.3 mm, vias 4 -> 2
- net D7: track 70.1 -> 79.2 mm, vias 2 -> 4
- net A1: track 65.4 -> 59.1 mm
- net SCL: track 83.5 -> 89.7 mm, vias 5 -> 3
- net D5: track 37.3 -> 42.4 mm, vias 2 -> 4
- net SCK: track 52.1 -> 48.1 mm, vias 4 -> 3
- net D6: track 17.0 -> 20.7 mm
- net GND: track 207.1 -> 203.5 mm, vias 8 -> 7
- net MISO: track 57.2 -> 53.9 mm, vias 3 -> 2
- net D10: track 34.3 -> 31.6 mm, vias 3 -> 1
- net D9: track 38.7 -> 36.1 mm
- net D2: track 70.5 -> 72.5 mm, vias 5 -> 3
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Other:
- board text added: "A0"

Commit message: update
Parts:
- moved C8 0.41 mm to (69.5, 15.8)
Other:
- board size 74.9 x 18 mm -> 74.6 x 18 mm
- board text added: "3.3"
- board text added: "RIFFLE-IT REV-D"
- board text added: "RIFFLE-ITO REV-D"
- board text added: "RST"
- board text added: "publiclab.org/wiki/riffle"
- board text removed: "RESET"
- board text removed: "RIFFLE-IT REV-F"
- board text removed: "RIFFLE-ITO REV-F"

Commit message: update
Changed lines of the file:
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@@
 <plain>
 <wire x1="0.0762" y1="-0.0762" x2="0.0762" y2="17.9324" width="0" layer="20"/>
-<wire x1="0.0762" y1="17.9324" x2="74.676" y2="17.9578" width="0" layer="20"/>
-<wire x1="74.676" y1="17.9578" x2="74.676" y2="-0.0508" width="0" layer="20"/>
-<wire x1="74.676" y1="-0.0508" x2="0.0762" y2="-0.0762" width="0" layer="20"/>
+<wire x1="0.0762" y1="17.9324" x2="74.6506" y2="17.907" width="0" layer="20"/>
+<wire x1="74.6506" y1="17.907" x2="74.6506" y2="-0.1016" width="0" layer="20"/>
+<wire x1="74.6506" y1="-0.1016" x2="0.0762" y2="-0.0762" width="0" layer="20"/>
 <text x="6.3754" y="4.953" size="0.6096" layer="21" rot="R270">ldo</text>
-<text x="39.3954" y="7.6962" size="0.6096" layer="21" rot="R270">EEPROM</text>
+<text x="39.2176" y="6.9088" size="0.6096" layer="21">EEPROM</text>
 <text x="22.606" y="13.6144" size="0.6096" layer="21">D6</text>
 <text x="28.702" y="14.2748" size="0.6096" layer="21" rot="R180">GND</text>
@@
 <text x="44.8818" y="5.461" size="0.6096" layer="21" rot="R270">D10</text>
 <text x="45.1866" y="8.3312" size="0.6096" layer="21" rot="R270">SCK</text>
-<text x="45.085" y="11.0744" size="0.6096" layer="21" rot="R270">MISO</text>
-<text x="51.7652" y="10.3378" size="0.6096" layer="21" rot="R270">D3</text>
+<text x="44.5516" y="11.0236" size="0.6096" layer="21" rot="R270">MISO</text>
+<text x="51.8668" y="10.5156" size="0.6096" layer="21" rot="R270">D3</text>
 <text x="51.7144" y="8.4074" size="0.6096" layer="21" rot="R270">MOSI</text>
 <text x="51.816" y="5.5372" size="0.6096" layer="21" rot="R270">D9</text>
-<text x="52.197" y="3.302" size="0.6096" layer="21" rot="R270">3.3V</text>
+<text x="51.7652" y="2.4384" size="0.6096" layer="21" rot="R270">3.3V</text>
 <text x="70.8406" y="17.399" size="0.6096" layer="21" rot="R270">3.3V</text>
 <text x="70.9168" y="9.5758" size="0.6096" layer="21" rot="R270">D2</text>
@@
 <text x="18.8468" y="9.5504" size="0.6096" layer="21" rot="R216">atmega328p</text>
 <text x="69.469" y="5.207" size="0.8128" layer="22" rot="MR0">publicab.org/wiki/riffle</text>
-<text x="70.231" y="0.889" size="0.8128" layer="21" rot="R90">RIFFLE-ITO REV-D</text>
+<text x="70.0532" y="0.889" size="0.8128" layer="21" rot="R90">RIFFLE-ITO REV-D</text>
 <text x="69.4182" y="6.1468" size="0.8128" layer="22" rot="MR0">RIFFLE-IT REV-D</text>
 <text x="69.4436" y="3.9624" size="0.8128" layer="22" rot="MR0">CERN OHL v1.2</text>
@@
 <wire x1="71.7296" y1="0.6858" x2="44.7294" y2="0.6604" width="0.4064" layer="22"/>
 <wire x1="44.7294" y1="0.6604" x2="44.7294" y2="15.24" width="0.4064" layer="22"/>
-<text x="66.548" y="12.7" size="0.8128" layer="22" rot="MR0">&lt;&lt;nordic RF24&gt;&gt;</text>
+<text x="66.3702" y="12.065" size="0.8128" layer="22" rot="MR0">&lt;&lt;nordic RF24&gt;&gt;</text>
 <text x="45.7454" y="3.2004" size="0.6096" layer="22" rot="MR270">GND</text>
 <wire x1="46.1264" y1="0.6604" x2="46.1264" y2="11.176" width="0.4064" layer="22"/>
@@
 <text x="19.558" y="13.6398" size="0.6096" layer="21">D3</text>
 <text x="70.866" y="4.3434" size="0.6096" layer="21" rot="R270">A0</text>
-<text x="68.4022" y="0.9144" size="0.8128" layer="21" rot="R90">publiclab.org/wiki/riffle</text>
+<text x="68.2498" y="0.9652" size="0.8128" layer="21" rot="R90">publiclab.org/wiki/riffle</text>
 <text x="14.9606" y="14.351" size="0.6096" layer="21" rot="R180">3.3</text>
 </plain>
@@
 </element>
 <element name="C8" library="resistor" package="C0805" value=".1u" x="69.4944" y="15.7988" smashed="yes" rot="R90">
-<attribute name="NAME" x="68.5038" y="17.3736" size="0.6096" layer="25" rot="R180"/>
+<attribute name="NAME" x="68.5292" y="17.399" size="0.6096" layer="25" rot="R180"/>
 <attribute name="VALUE" x="71.7804" y="14.9098" size="1.27" layer="27" rot="R90"/>
 </element>
@@
 </element>
 <element name="CRF" library="resistor" package="C0805" value="100u" x="43.3832" y="2.1082" smashed="yes" rot="R180">
-<attribute name="NAME" x="44.5008" y="1.0922" size="0.6096" layer="25" rot="R180"/>
+<attribute name="NAME" x="44.6532" y="3.683" size="0.6096" layer="25" rot="R180"/>
 <attribute name="VALUE" x="44.2722" y="4.3942" size="1.27" layer="27" rot="R180"/>
 </element>
