File: hardware/riffleito-REVD.brd (EAGLE design)
At the start: 74.6 x 18 mm, 31 parts, among them IC1 ATMEGA328P, IC2 24AA128SN, IC4 MCP1700-33, X1 16 MHz

Commit message: update
Parts:
- CRF: value 100u -> .1u
Changed lines of the file:
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@@
 <text x="69.4182" y="6.1468" size="0.8128" layer="22" rot="MR0">RIFFLE-IT REV-D</text>
 <text x="69.4436" y="3.9624" size="0.8128" layer="22" rot="MR0">CERN OHL v1.2</text>
-<wire x1="44.704" y1="15.4432" x2="71.9074" y2="15.3924" width="0.4064" layer="22"/>
-<wire x1="71.7296" y1="0.6858" x2="44.7294" y2="0.6604" width="0.4064" layer="22"/>
-<wire x1="44.7294" y1="0.6604" x2="44.7294" y2="15.24" width="0.4064" layer="22"/>
+<wire x1="45.1866" y1="15.3924" x2="71.9074" y2="15.3924" width="0.4064" layer="22"/>
+<wire x1="71.7296" y1="0.6858" x2="45.2374" y2="0.6604" width="0.4064" layer="22"/>
 <text x="66.3702" y="12.065" size="0.8128" layer="22" rot="MR0">&lt;&lt;nordic RF24&gt;&gt;</text>
 <text x="45.7454" y="3.2004" size="0.6096" layer="22" rot="MR270">GND</text>
@@
 <text x="68.2498" y="0.9652" size="0.8128" layer="21" rot="R90">publiclab.org/wiki/riffle</text>
 <text x="14.9606" y="14.351" size="0.6096" layer="21" rot="R180">3.3</text>
+<wire x1="45.3644" y1="15.367" x2="45.1866" y2="15.367" width="0.4064" layer="22"/>
+<wire x1="45.1866" y1="15.367" x2="45.1866" y2="3.683" width="0.4064" layer="22"/>
 </plain>
 <attributes>
@@
 <attribute name="VALUE" x="40.5638" y="18.5166" size="1.27" layer="27" rot="R180"/>
 </element>
-<element name="CRF" library="resistor" package="C0805" value="100u" x="43.3832" y="2.1082" smashed="yes" rot="R180">
+<element name="CRF" library="resistor" package="C0805" value=".1u" x="43.3832" y="2.1082" smashed="yes" rot="R180">
 <attribute name="NAME" x="44.6532" y="3.683" size="0.6096" layer="25" rot="R180"/>
 <attribute name="VALUE" x="44.2722" y="4.3942" size="1.27" layer="27" rot="R180"/>
