File: hardware/conduct-555-2.brd (EAGLE design)
At the start: 33.2 x 17.8 mm, 15 parts, among them J2 AYZ0202

Commit message: update
Parts:
- moved C2 1.27 mm to (18.5, 7.62)
- moved C1 1.27 mm to (15.0, 7.62)
- moved C7 1.08 mm to (22.1, 7.62)
Changed lines of the file:
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@@
 <element name="555" library="SparkFun-AnalogIC" package="SO08@1" value="NE555D" x="8.636" y="14.732" rot="R270"/>
 <element name="J2" library="SparkFunNew" package="AYZ0202" value="AYZ0202" x="7.874" y="4.064" rot="R90"/>
-<element name="C1" library="resistor" package="C0805" value="1uF" x="13.97" y="6.858" rot="R270"/>
-<element name="C2" library="resistor" package="C0805" value=".1uF" x="17.526" y="6.858" rot="R270"/>
+<element name="C1" library="resistor" package="C0805" value="1uF" x="14.986" y="7.62" rot="R270"/>
+<element name="C2" library="resistor" package="C0805" value=".1uF" x="18.542" y="7.62" rot="R270"/>
 <element name="C3" library="resistor" package="C0805" value=".01u" x="10.922" y="10.414" rot="R180"/>
 <element name="R1" library="rcl" package="R0805" value="3.3K" x="15.748" y="16.002" rot="R180"/>
@@
 <element name="C5" library="resistor" package="C0805" value="100n" x="21.082" y="16.002" rot="R180"/>
 <element name="C6" library="resistor" package="C0805" value=".1uF" x="20.828" y="12.446" rot="R180"/>
-<element name="C7" library="resistor" package="C0805" value="1uF" x="21.336" y="6.858" rot="R270"/>
+<element name="C7" library="resistor" package="C0805" value="1uF" x="22.098" y="7.62" rot="R270"/>
 <element name="JP2" library="SparkFun-Connectors" package="1X05" value="" x="13.208" y="1.27" smashed="yes">
 <attribute name="VALUE" x="11.938" y="-1.905" size="1.27" layer="27"/>
@@
 <wire x1="21.678" y1="12.446" x2="21.932" y2="16.002" width="0" layer="19" extent="1-1"/>
 <wire x1="16.698" y1="12.446" x2="21.678" y2="12.446" width="0" layer="19" extent="1-1"/>
-<wire x1="21.336" y1="7.708" x2="21.678" y2="12.446" width="0" layer="19" extent="1-1"/>
-<wire x1="11.772" y1="10.414" x2="21.336" y2="7.708" width="0" layer="19" extent="1-1"/>
-<wire x1="13.97" y1="6.008" x2="11.772" y2="10.414" width="0" layer="19" extent="1-1"/>
-<wire x1="17.526" y1="6.008" x2="16.698" y2="12.446" width="0" layer="19" extent="1-1"/>
-<wire x1="7.2" y1="10.414" x2="17.526" y2="6.008" width="0" layer="19" extent="1-1"/>
+<wire x1="22.098" y1="8.47" x2="21.678" y2="12.446" width="0" layer="19" extent="1-1"/>
+<wire x1="11.772" y1="10.414" x2="22.098" y2="8.47" width="0" layer="19" extent="1-1"/>
+<wire x1="14.986" y1="6.77" x2="11.772" y2="10.414" width="0" layer="19" extent="1-1"/>
+<wire x1="18.542" y1="6.77" x2="16.698" y2="12.446" width="0" layer="19" extent="1-1"/>
+<wire x1="7.2" y1="10.414" x2="18.542" y2="6.77" width="0" layer="19" extent="1-1"/>
 <wire x1="6.0198" y1="16.637" x2="7.2" y2="10.414" width="0" layer="19" extent="1-1"/>
 <wire x1="1.27" y1="1.27" x2="7.2" y2="10.414" width="0" layer="19" extent="1-1"/>
@@
 <contactref element="J2" pad="4"/>
 <contactref element="C1" pad="1"/>
-<wire x1="10.699" y1="1.564" x2="13.97" y2="7.708" width="0" layer="19" extent="1-1"/>
+<wire x1="10.699" y1="1.564" x2="14.986" y2="8.47" width="0" layer="19" extent="1-1"/>
 <wire x1="5.049" y1="1.564" x2="10.699" y2="1.564" width="0" layer="19" extent="1-1"/>
 </signal>
@@
 <contactref element="J2" pad="6"/>
 <contactref element="C2" pad="1"/>
-<wire x1="10.699" y1="6.564" x2="17.526" y2="7.708" width="0" layer="19" extent="1-1"/>
+<wire x1="10.699" y1="6.564" x2="18.542" y2="8.47" width="0" layer="19" extent="1-1"/>
 <wire x1="5.049" y1="6.564" x2="10.699" y2="6.564" width="0" layer="19" extent="1-1"/>
 </signal>

Commit message: update
Parts:
- removed J-EC, J-THRM: 1X2-3.5MM, adafruit:1X2-3.5MM
- added EC, THRM: 1X2-3.5MM, adafruit:1X2-3.5MM
- moved JP2 4.07 mm to (17.3, 1.40)
- moved C7 3.84 mm to (25.9, 8.13)
- moved C2 3.84 mm to (22.4, 8.13)
- moved C1 3.59 mm to (18.5, 8.13)
- moved C6 3.57 mm to (24.4, 12.7)
- moved R2 3.44 mm to (19.2, 12.7)
- moved R1 3.31 mm to (19.1, 16.3)
- moved C5 3.31 mm to (24.4, 16.3)
- moved C3 2.93 mm to (13.8, 10.7)
- moved C4 2.68 mm to (9.02, 10.7)
- moved J2 2.43 mm to (10.3, 4.32), turned to 270 degrees
- moved 555 1.78 mm to (10.4, 14.7)
- moved JP4 0.18 mm to (1.40, 1.40)
Connections:
- net N$3: now also EC.1; no longer J-EC.1
- net N1: now also EC.2; no longer J-EC.2
- net THRM: now also THRM.1; no longer J-THRM.1
- net VCC: now also C4.2, C5.2, C6.2, C7.2, THRM.2; no longer J-THRM.2
Routing:
- net GND: track 0.00 -> 72.3 mm
- net VCC: track 0.00 -> 68.0 mm
- net N1: track 0.00 -> 58.3 mm, vias 0 -> 2
- net THRM: track 0.00 -> 37.2 mm, vias 0 -> 3
- net SCL: track 0.00 -> 32.0 mm, vias 0 -> 1
- net SDA: track 0.00 -> 29.6 mm, vias 0 -> 1
- net N$3: track 0.00 -> 25.3 mm, vias 0 -> 1
- net A1: track 0.00 -> 21.4 mm, vias 0 -> 1
- net N$6: track 0.00 -> 18.0 mm, vias 0 -> 2
- net VDD2: track 0.00 -> 13.2 mm
- net EC: track 0.00 -> 8.64 mm, vias 0 -> 1
- net N$2: track 0.00 -> 2.22 mm
Other:
- board size 33.2 x 17.8 mm -> 36.8 x 18 mm
- board text added: "1"
- board text added: "2"
- board text added: "3.3"
- board text added: "555"
- board text added: "A1"
- board text added: "CERN OHL v1.2"
- board text added: "EC"
- board text added: "GND"
- board text added: "REV-A"
- board text added: "RIFF-CT"
- board text added: "RIFF-CT-REVA"
- board text added: "SCL"
- board text added: "SDA"
- board text added: "THM"
- board text added: "conductivity + temperature"
- board text added: "publiclab.org/wiki/riffle"

Commit message: update
Parts:
- moved JP2 0.63 mm to (16.6, 1.40)
- moved J2 0.13 mm to (10.2, 4.32)
Connections:
- net GND: now also THRM.1; no longer R2.1
- net THRM: now also R2.1, THRM.2; no longer R2.2, THRM.1
- net VCC: now also R2.2; no longer THRM.2
Routing:
- net GND: track 72.3 -> 81.0 mm, vias 0 -> 2
- net N$3: track 25.3 -> 33.4 mm
- net SCL: track 32.0 -> 27.2 mm
- net VCC: track 68.0 -> 72.3 mm, vias 0 -> 1
- net THRM: track 37.2 -> 41.2 mm, vias 3 -> 2
- net EC: track 8.64 -> 11.4 mm
- net N1: track 58.3 -> 60.2 mm
- net N$6: track 18.0 -> 19.6 mm
- net SDA: track 29.6 -> 29.1 mm
Other:
- board text added: "RIFFLE-CT"
- board text added: "RIFFLE-CT-REVA"
- board text removed: "REV-A"
- board text removed: "RIFF-CT"
- board text removed: "RIFF-CT-REVA"
