File: hardware/riffleito-REVD.sch (EAGLE design)
At the start: 29 parts, among them IC1 ATMEGA328P, IC2 24AA128SN, IC4 MCP1700-33, X1 16 MHz

Commit message: routed!
Connections:
- net A0: now also SENSE.4; no longer SENSE.5
- net A1: now also SENSE.5; no longer SENSE.6
- net GND: now also SENSE.1; no longer SENSE.4
- net SCL: now also SENSE.2; no longer SENSE.1
- net SDA: now also SENSE.3; no longer SENSE.2
- net VCC: now also SENSE.6; no longer SENSE.3
Other:
- moved on the sheet: SENSE
Changed lines of the file:
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@@
 <instance part="P+4" gate="VCC" x="-156.21" y="1.27"/>
 <instance part="P+10" gate="VCC" x="-140.97" y="1.27"/>
-<instance part="SENSE" gate="G$1" x="-51.816" y="-7.366" rot="R180"/>
+<instance part="SENSE" gate="G$1" x="-51.308" y="-7.366" rot="R180"/>
 <instance part="FTDI" gate="G$1" x="-73.914" y="93.98" rot="R180"/>
 <instance part="RAD" gate="G$1" x="176.53" y="93.98" rot="R180"/>
@@
 <wire x1="-92.202" y1="15.748" x2="-88.9" y2="15.748" width="0.1524" layer="91"/>
 <pinref part="C8" gate="G$1" pin="1"/>
-</segment>
-<segment>
-<wire x1="-56.896" y1="-9.906" x2="-67.056" y2="-9.906" width="0.1524" layer="91"/>
-<wire x1="-67.056" y1="-9.906" x2="-67.056" y2="-10.16" width="0.1524" layer="91"/>
-<label x="-70.358" y="-10.16" size="1.778" layer="95"/>
-<pinref part="SENSE" gate="G$1" pin="4"/>
 </segment>
 <segment>
@@
 <pinref part="GND1" gate="1" pin="GND"/>
 </segment>
+<segment>
+<wire x1="-56.388" y1="-2.286" x2="-67.564" y2="-2.286" width="0.1524" layer="91"/>
+<label x="-69.596" y="-1.524" size="1.778" layer="95"/>
+<pinref part="SENSE" gate="G$1" pin="1"/>
+</segment>
 </net>
 <net name="A0" class="0">
@@
 </segment>
 <segment>
-<wire x1="-56.896" y1="-12.446" x2="-69.342" y2="-12.446" width="0.1524" layer="91"/>
-<wire x1="-69.342" y1="-12.446" x2="-69.342" y2="-11.938" width="0.1524" layer="91"/>
-<label x="-73.152" y="-12.446" size="1.778" layer="95"/>
-<pinref part="SENSE" gate="G$1" pin="5"/>
+<wire x1="-56.388" y1="-9.906" x2="-67.056" y2="-9.906" width="0.1524" layer="91"/>
+<wire x1="-67.056" y1="-9.906" x2="-67.056" y2="-10.16" width="0.1524" layer="91"/>
+<label x="-70.358" y="-10.16" size="1.778" layer="95"/>
+<pinref part="SENSE" gate="G$1" pin="4"/>
 </segment>
 </net>
@@
 <wire x1="-78.232" y1="15.748" x2="-80.01" y2="15.748" width="0.1524" layer="91"/>
 <wire x1="-80.01" y1="15.748" x2="-81.28" y2="15.748" width="0.1524" layer="91"/>
-<wire x1="-80.01" y1="15.748" x2="-80.01" y2="-7.366" width="0.1524" layer="91"/>
-<wire x1="-80.01" y1="-7.366" x2="-56.896" y2="-7.366" width="0.1524" layer="91"/>
+<wire x1="-80.01" y1="15.748" x2="-80.01" y2="-15.24" width="0.1524" layer="91"/>
 <junction x="-80.01" y="15.748"/>
 <pinref part="C8" gate="G$1" pin="2"/>
-<pinref part="SENSE" gate="G$1" pin="3"/>
+<pinref part="SENSE" gate="G$1" pin="6"/>
+<wire x1="-80.01" y1="-15.24" x2="-56.896" y2="-15.24" width="0.1524" layer="91"/>
+<wire x1="-56.896" y1="-15.24" x2="-56.388" y2="-14.986" width="0.1524" layer="91"/>
 </segment>
 <segment>
@@
 </segment>
 <segment>
-<wire x1="-56.896" y1="-14.986" x2="-70.358" y2="-14.986" width="0.1524" layer="91"/>
-<label x="-74.93" y="-15.494" size="1.778" layer="95"/>
-<pinref part="SENSE" gate="G$1" pin="6"/>
+<wire x1="-56.388" y1="-12.446" x2="-69.342" y2="-12.446" width="0.1524" layer="91"/>
+<wire x1="-69.342" y1="-12.446" x2="-69.342" y2="-11.938" width="0.1524" layer="91"/>
+<label x="-73.152" y="-12.446" size="1.778" layer="95"/>
+<pinref part="SENSE" gate="G$1" pin="5"/>
 </segment>
 </net>
@@
 <net name="SDA" class="0">
 <segment>
-<wire x1="-56.896" y1="-4.826" x2="-67.056" y2="-4.826" width="0.1524" layer="91"/>
-<label x="-70.866" y="-4.318" size="1.778" layer="95"/>
-<pinref part="SENSE" gate="G$1" pin="2"/>
-</segment>
-<segment>
 <pinref part="IC1" gate="G$1" pin="PC4(ADC4/SDA)"/>
 <wire x1="62.23" y1="52.07" x2="67.056" y2="52.07" width="0.1524" layer="91"/>
@@
 <label x="-140.208" y="-16.256" size="1.778" layer="95"/>
 </segment>
+<segment>
+<pinref part="SENSE" gate="G$1" pin="3"/>
+<wire x1="-56.388" y1="-7.366" x2="-66.802" y2="-7.366" width="0.1524" layer="91"/>
+<label x="-71.882" y="-7.366" size="1.778" layer="95"/>
+</segment>
 </net>
 <net name="SCL" class="0">
-<segment>
-<wire x1="-56.896" y1="-2.286" x2="-67.564" y2="-2.286" width="0.1524" layer="91"/>
-<label x="-69.596" y="-1.524" size="1.778" layer="95"/>
-<pinref part="SENSE" gate="G$1" pin="1"/>
-</segment>
 <segment>
 <pinref part="IC1" gate="G$1" pin="PC5(ADC5/SCL)"/>
@@
 <label x="-154.94" y="-15.748" size="1.778" layer="95"/>
 </segment>
-</net>
+<segment>
+<pinref part="SENSE" gate="G$1" pin="2"/>
+<wire x1="-56.388" y1="-4.826" x2="-67.564" y2="-4.826" width="0.1524" layer="91"/>
+<label x="-72.644" y="-4.826" size="1.778" layer="95"/>
+</segment>
+</net>

Commit message: update
Changed lines of the file:
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@@
 </instance>
 <instance part="X1" gate="G$1" x="10.16" y="41.91" rot="R270"/>
-<instance part="P+11" gate="G$1" x="-21.59" y="77.47"/>
+<instance part="P+11" gate="G$1" x="-19.812" y="77.47"/>
 <instance part="C7" gate="G$1" x="-29.21" y="62.23" smashed="yes" rot="R90">
 <attribute name="NAME" x="-31.496" y="60.071" size="1.778" layer="95"/>
@@
 </segment>
 <segment>
-<wire x1="-21.59" y1="77.47" x2="-21.59" y2="74.93" width="0.1524" layer="91"/>
+<wire x1="-19.812" y1="77.47" x2="-21.59" y2="74.93" width="0.1524" layer="91"/>
 <pinref part="P+11" gate="G$1" pin="3.3V"/>
 <pinref part="RRST" gate="G$1" pin="1"/>
@@
 </segment>
 </net>
-<net name="N$4" class="0">
-<segment>
-<wire x1="-13.716" y1="-40.64" x2="-13.716" y2="-40.386" width="0.1524" layer="91"/>
-</segment>
-</net>

Commit message: update
Parts:
- removed C9: .1uF, rcl:C-EUC0805
- removed FTDI, SENSE: (no value), SparkFun-Connectors:M06SIP
- removed RAD: M04X2, SparkFun-Connectors:M04X2
- added CRF: 100u, resistor:C-EUC0805
- added CSD: .1uF, resistor:C-EUC0805
- added JP1: (no value), SparkFun-Connectors:M081X08
- added JP4: (no value), SparkFun-Connectors:M07
- added RTCINT: SOLDERJUMPERNO, _SparkFun:SOLDERJUMPERNO
- added U$1: M04X2, SparkFun-Connectors:M04X2
- JP2: device SparkFun-Connectors:M07 -> SparkFun-Connectors:M06SIP
Connections:
- new net N$1: RRTC1.2, RTC.INT/SQW, RTCINT.1
- new net N$4: JP4.7, REMOTE.D
- net A0: now also JP4.2; no longer SENSE.4
- net A1: now also JP4.3; no longer SENSE.5
- net A2: now also JP1.4; no longer JP2.4
- net D10: now also U$1.6; no longer RAD.3
- net D2: now also JP4.4; no longer FTDI.5
- net D3: now also JP1.5, RTCINT.2, U$1.1; no longer RAD.4
- net D6: now also JP1.6; no longer JP2.5
- net D8: now also JP1.7; no longer JP2.6
- net D9: now also U$1.5; no longer RRTC1.2, RTC.INT/SQW
- net DTR: now also JP2.1; no longer FTDI.1
- net GND: now also CRF.2, CSD.2, JP1.8, JP2.5, JP2.6, JP4.1, U$1.8; no longer C9.1, FTDI.6, JP2.7, RAD.1, SENSE.1
- net MISO: now also U$1.2; no longer RAD.7
- net MOSI: now also U$1.3; no longer RAD.6
- net RESET: now also JP1.2; no longer JP2.2
- net RXD: now also JP2.3; no longer FTDI.3
- net SCK: now also U$1.4; no longer RAD.5
- net SCL: now also JP4.6; no longer SENSE.2
- net SDA: now also JP4.5; no longer SENSE.3
- net TXD: now also JP2.2; no longer FTDI.2
- net VCC: now also CRF.1, JP1.3, U$1.7; no longer C8.2, JP2.3, RAD.2, REMOTE.D, SENSE.6
- net VDD: now also CSD.1; no longer C9.2
- net VIN: now also JP1.1, JP2.4; no longer FTDI.4, JP2.1
Other:
- moved on the sheet: C8, RRTC1

Commit message: update
Connections:
- net N$4: now also C8.2
Other:
- moved on the sheet: C8
Changed lines of the file:
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@@
 <instance part="GND2" gate="1" x="-94.742" y="15.748" rot="R270"/>
 <instance part="P+2" gate="VCC" x="-62.484" y="18.288"/>
-<instance part="C8" gate="G$1" x="-87.122" y="16.002" smashed="yes" rot="R90">
-<attribute name="NAME" x="-87.503" y="17.526" size="1.778" layer="95" rot="R90"/>
-<attribute name="VALUE" x="-84.201" y="22.098" size="1.778" layer="96" rot="R270"/>
+<instance part="C8" gate="G$1" x="-87.884" y="15.748" smashed="yes" rot="R90">
+<attribute name="NAME" x="-88.265" y="17.272" size="1.778" layer="95" rot="R90"/>
+<attribute name="VALUE" x="-84.963" y="21.844" size="1.778" layer="96" rot="R270"/>
 </instance>
 <instance part="RTC" gate="G$1" x="133.35" y="-12.7"/>
@@
 <segment>
 <pinref part="GND2" gate="1" pin="GND"/>
-<wire x1="-92.202" y1="15.748" x2="-89.662" y2="16.002" width="0.1524" layer="91"/>
+<wire x1="-92.202" y1="15.748" x2="-90.424" y2="15.748" width="0.1524" layer="91"/>
 <pinref part="C8" gate="G$1" pin="1"/>
 </segment>
@@
 <wire x1="-79.502" y1="-18.034" x2="-55.88" y2="-18.034" width="0.1524" layer="91"/>
 <wire x1="-55.88" y1="-18.034" x2="-55.88" y2="-17.526" width="0.1524" layer="91"/>
-</segment>
-</net>
+<pinref part="C8" gate="G$1" pin="2"/>
+<wire x1="-79.502" y1="15.748" x2="-82.804" y2="15.748" width="0.1524" layer="91"/>
+<junction x="-79.502" y="15.748"/>
+</segment>
+</net>

Commit message: update
Parts:
- CRF: value 100u -> .1u
Changed lines of the file:
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@@
 <setting verticaltext="up"/>
 </settings>
-<grid distance="0.01" unitdist="inch" unit="inch" style="lines" multiple="1" display="no" altdistance="0.01" altunitdist="inch" altunit="inch"/>
+<grid distance="0.1" unitdist="inch" unit="inch" style="lines" multiple="1" display="no" altdistance="0.01" altunitdist="inch" altunit="inch"/>
 <layers>
 <layer number="1" name="Top" color="4" fill="1" visible="no" active="no"/>
@@
 <part name="P+3" library="supply1" deviceset="VCC" device=""/>
 <part name="GND1" library="supply1" deviceset="GND" device=""/>
-<part name="CRF" library="resistor" deviceset="C-EU" device="C0805" value="100u"/>
+<part name="CRF" library="resistor" deviceset="C-EU" device="C0805" value=".1u"/>
 <part name="GND6" library="supply1" deviceset="GND" device=""/>
 <part name="P+12" library="supply1" deviceset="VCC" device=""/>
